Commit message: Add suction gripper

File: panda_arm.urdf (robot description, URDF)
Before this commit: robot panda, 9 links, 8 joints
Links:
- added link panda_eef; collision mesh filename=package://franka_description/meshes/collision/gripper.stl; visual mesh filename=package://franka_description/meshes/visual/gripper.stl
- added link panda_tip
Joints:
- added joint panda_joint_eef: type fixed, parent panda_link8, child panda_eef, origin xyz=0 0 0 rpy=0 0 0
- added joint panda_joint_tip: type fixed, parent panda_eef, child panda_tip, origin xyz=0 0 0.04 rpy=0 1.57 0
- joint panda_joint1: limit lower=-2.8973 upper=2.8973 effort=87 velocity=2.1750 -> lower=-2.8973 upper=2.8973 effort=0 velocity=0
- joint panda_joint2: limit lower=-1.7628 upper=1.7628 effort=87 velocity=2.1750 -> lower=-1.7628 upper=1.7628 effort=0 velocity=0
- joint panda_joint3: limit lower=-2.8973 upper=2.8973 effort=87 velocity=2.1750 -> lower=-2.8973 upper=2.8973 effort=0 velocity=0
- joint panda_joint4: limit lower=-3.0718 upper=-0.0698 effort=87 velocity=2.1750 -> lower=-3.0718 upper=-0.0698 effort=0 velocity=0
- joint panda_joint5: limit lower=-2.8973 upper=2.8973 effort=12 velocity=2.6100 -> lower=-2.8973 upper=2.8973 effort=0 velocity=0
- joint panda_joint6: limit lower=-0.0175 upper=3.7525 effort=12 velocity=2.6100 -> lower=-0.0175 upper=3.7525 effort=0 velocity=0
- joint panda_joint7: limit lower=-2.8973 upper=2.8973 effort=12 velocity=2.6100 -> lower=-2.8973 upper=2.8973 effort=0 velocity=0
